File: MicroPro-RP2040.kicad_sch (KiCad schematic)
At the start: 55 parts, among them J1 USB_C_Receptacle_USB2.0_16P, J2 Qwiic, J3 Conn_02x12_Counter_Clockwise, J4 Conn_01x04, SW1 Boot, SW2 Reset, U1 RP2040, U2 AP2112K-3.3, U3 W25Q128JV, U5 TMUX1204DQAR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

Commit message: completed schematics, generated BOM
Parts:
- C1, C2: Comments (none) -> C0G dielectric
- C21: value ~ -> 1.5n; Comments (none) -> C0G dielectric
- D1: Manufacturer_Part_Number (none) -> PMEG2005EJ-QX
- F1: Manufacturer_Part_Number (none) -> SMD0603B050TF
- J2: Manufacturer_Part_Number (none) -> SM04B-SRSS-TB(LF)(SN)(P)
- R8: value ~ -> 1.47k
- R9: value ~ -> 24.9
- RN1: Manufacturer_Part_Number (none) -> EXB-V4V270JV
- RN2: Manufacturer_Part_Number CAT16-1003F4LF -> CAT16-1002F4LF
- U2: Manufacturer_Part_Number (none) -> AP2112K-3.3TRG1
- U3: Manufacturer_Part_Number (none) -> W25Q128JVPIM
- U6: value ADS7044IRUGR -> ADS7042IRUGR; Manufacturer_Part_Number ADS7044IRUGR -> ADS7042IRUGR; Mouser Part Number 595-ADS7044IRUGR -> (none); Mouser Price/Stock https://www.mouser.co.uk/ProductDetail/Texas-Instruments/AD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 -> (none)
- U7: Manufacturer_Part_Number (none) -> LM4040A30IDCKR
- Y1: Manufacturer_Part_Number (none) -> ABM8-272-T3
