File: MicroPro-RP2040.kicad_pcb (KiCad board)
At the start: 4 copper layers, 40 x 50 mm, 55 parts, among them J1 USB_C_Receptacle_USB2.0_16P, J2 Qwiic, J3 Conn_02x12_Counter_Clockwise, J4 Conn_01x04, SW1 Boot, SW2 Reset, U1 RP2040, U2 AP2112K-3.3, U3 W25Q128JV, U5 TMUX1204DQAR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

Commit message: v1.0 board
Parts:
- added G***: LOGO, MicroPro:open-source-hardware-logo-no-text, B.Cu at (111.8, 101.6)
- C21: value ~ -> 1.5n
- R8: value ~ -> 1.47k
- R9: value ~ -> 24.9
- U6: value ADS7044IRUGR -> ADS7042IRUGR
Routing:
- net /usb-: track 1.79 -> 13.4 mm
- net /usb+: track 1.92 -> 13.3 mm
- net /D+: track 4.16 -> 10.7 mm
- net /D-: track 5.59 -> 9.99 mm
- net GND: track 4.45 -> 5.81 mm
Other:
- board text added: "v1.0"

Commit message: optimized via position
Routing:
- net +3V3: track 37.2 -> 38.5 mm
- net 18/A0: track 20.4 -> 21.3 mm
- net 19/A1: track 18.3 -> 19.2 mm
- net BOOT: track 14.2 -> 15.1 mm
- net VBUS: track 14.1 -> 14.7 mm

Commit message: fixed miswiring in schematics, v1.1 board
Connections:
- net 0 renamed GP0
- net 1 renamed GP1
- net 2 renamed GP2
- net 20 renamed GP20
- net 21 renamed GP21
- net 22 renamed GP22
- net 23 renamed GP23
- net 26 renamed GP26
- net 27 renamed GP27
- net 28 renamed GP28
- net 29 renamed GP29
- net 3 renamed GP3
- net 4 renamed GP4
- net 5 renamed GP5
- net 6 renamed GP6
- net 7 renamed GP7
- net 8 renamed GP8
- net 9 renamed GP9
- J2 pad 3: 16 -> 16/SDA
- J2 pad 4: 17 -> 17/SCL
- RN2 pad 3: 16 -> 17/SCL
- RN2 pad 5: 17 -> 16/SDA
- U1 pad 27: 17 -> 16/SDA
- U1 pad 28: 16 -> 17/SCL
Routing:
- net 16: track 18.0 -> 0.00 mm
- net 17/SCL: track 0.00 -> 16.5 mm
- net 16/SDA: track 0.00 -> 10.7 mm
- net 17: track 8.83 -> 0.00 mm
Other:
- board text added: "v1.1"
- board text removed: "v1.0"

Commit message: generated gerber, added license, readme
Connections:
- U3 pad 9: (no net) -> GND
Routing:
- net GND: vias 18 -> 19
